File: ACS PCB.kicad_sch (KiCad schematic)
At the start: 10 parts, among them U2 TPSM84338RCJR

Commit message: i-added-hello
Other:
- note added: "HELLOOOO"
Changed lines of the file:
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@@
+		)
+	)
+	(text "HELLOOOO"
+		(exclude_from_sim no)
+		(at 78.105 118.11 0)
+		(effects
+			(font
+				(size 1.27 1.27)
+			)
 		)
 	)

Commit message: added-more-hierarchical-boxes
Parts:
- removed C1, C2: 10u, Capacitor_SMD:C_0603_1608Metric, symbol Device:C
- removed C3, C6: 100n, Capacitor_SMD:C_0603_1608Metric, symbol Device:C
- removed C4, C5: 22u, Capacitor_SMD:C_0603_1608Metric, symbol Device:C
- removed R1: 30k, Resistor_SMD:R_0603_1608Metric, symbol Device:R_US
- removed R2: 220k, Resistor_SMD:R_0603_1608Metric, symbol Device:R_US
- removed U2: TPSM84338RCJR, RCJ0009A-MFG, symbol TPSM84338RCJR:TPSM84338RCJR
Connections:
- no-connect marks 6 -> 1
Other:
- added sheet LED indicator (LEDindicator.kicad_sch)
- added sheet Power (power.kicad_sch)
- added sheet WiFi board (WiFiboard.kicad_sch)
- note removed: "HELLOOOO"
- note removed: "apparently ts bad :("
- note removed: "should be >25V rated capacitors"
- note removed: "things to add: - wifi board - indicater led light"
