File: ACS PCB.kicad_sch (KiCad schematic)
At the start: 1 part

Commit message: finished voltage converter i think :sob: ugh ugh ughgit add .git add .
Connections:
- net VoltMonitor: now reaches A1.D28
- net Vin renamed 5V
Other:
- removed sheet WiFi board
Changed lines of the file:
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@@
 	(text "interrupts? maybe? no?"
 		(exclude_from_sim no)
-		(at 226.695 84.455 0)
+		(at 246.38 73.025 0)
 		(effects
 			(font
@@
 	(wire
 		(pts
+			(xy 212.09 66.04) (xy 224.155 66.04)
+		)
+		(stroke
+			(width 0)
+			(type default)
+		)
+	)
+	(wire
+		(pts
 			(xy 212.09 71.12) (xy 224.79 71.12)
 		)
@@
 		)
 	)
-	(global_label "Vin"
+	(global_label "5V"
 		(shape input)
 		(at 219.075 33.02 0)
@@
 		)
 		(property "Intersheetrefs" "${INTERSHEET_REFS}"
-			(at 224.9026 33.02 0)
+			(at 224.3583 33.02 0)
+			(hide yes)
+			(show_name no)
+			(do_not_autoplace no)
+			(effects
+				(font
+					(size 1.27 1.27)
+				)
+				(justify left)
+			)
+		)
+	)
+	(global_label "VoltMonitor"
+		(shape input)
+		(at 224.155 66.04 0)
+		(fields_autoplaced yes)
+		(effects
+			(font
+				(size 1.27 1.27)
+			)
+			(justify left)
+		)
+		(property "Intersheetrefs" "${INTERSHEET_REFS}"
+			(at 237.7838 66.04 0)
 			(hide yes)
 			(show_name no)
@@
 	)
 	(sheet
-		(at 38.735 28.575)
+		(at 62.23 40.005)
 		(size 61.595 36.195)
 		(exclude_from_sim no)
@@
 		)
 		(property "Sheetname" "Power"
-			(at 38.735 27.8634 0)
+			(at 62.23 39.2934 0)
 			(show_name no)
 			(do_not_autoplace no)
@@
 		)
 		(property "Sheetfile" "power.kicad_sch"
-			(at 38.735 65.3546 0)
+			(at 62.23 76.7846 0)
 			(show_name no)
 			(do_not_autoplace no)
@@
 				)
 			)
-		)
-	)
-	(sheet
-		(at 100.965 112.395)
-		(size 51.435 35.56)
-		(exclude_from_sim no)
-		(in_bom yes)
-		(on_board yes)
-		(dnp no)
-		(fields_autoplaced yes)
-		(stroke
-			(width 0.1524)
-			(type solid)
-		)
-		(fill
-			(color 0 0 0 0)
-		)
-		(property "Sheetname" "WiFi board"
-			(at 100.965 111.6834 0)
-			(show_name no)
-			(do_not_autoplace no)
-			(effects
-				(font
-					(size 1.27 1.27)
-				)
-				(justify left bottom)
-			)
-		)
-		(property "Sheetfile" "WiFiboard.kicad_sch"
-			(at 100.965 148.5396 0)
-			(show_name no)
-			(do_not_autoplace no)
-			(effects
-				(font
-					(size 1.27 1.27)
-				)
-				(justify left top)
-			)
-		)
-		(instances
-			(project "ACS PCB"
-				(path "/67a598cb-afc0-4277-b58a-8f35d31efc48"
-					(page "5")
-				)
-			)

Commit message: Fixed symbols and ran ERC
Parts:
- added J5: Conn_01x02, symbol Connector_Generic:Conn_01x02
Connections:
- net GND: now also J5.2 (Pin_2)
- net CS_A0: now reaches A1.D10 ((CS)D10)
- net CS_A1: now reaches A1.D14 (A0)
- net CS_I1: now reaches A1.D15 (A1)
- net CS_A2: now reaches A1.D16 (A2)
- net CS_I2: now reaches A1.D17 (A3)
- net PWM_fs: now reaches A1.D24 (A10)
- net PWM_ss: now reaches A1.D25 (A11)
- net MISO1: now reaches A1.D26 (A12)
- net SCK1: now reaches A1.D27 (A13)
- net INT_I2: now reaches A1.D29
- net INT_A0: now reaches A1.D36
- net INT_I0: now reaches A1.D37
- net MOSI1: now reaches A1.D39 (A15)
- net 3.3V renamed +3.3V
- net CS1: no longer names the net of A1.D4
- net CS3: no longer names the net of A1.D3
- net CS4 renamed CS_I0
- net CS5: no longer names the net of A1.D6
- net CS6: no longer names the net of A1.D5
- net CS7: no longer names the net of A1.D2
- net INT1 renamed INT_A1
- net INT3 renamed INT_I1
- net INT7 renamed INT_A2
- net SCK renamed SCK0
- net SDI renamed MOSI0
- net SDO renamed MISO0
- new net +BATT: J5.1 (Pin_1)
- no-connect marks 1 -> 22
Other:
- added sheet Motor Interfacing (motorInterfacing.kicad_sch)
- note added: "Alt/IMU 0 / Alt 2 --> SPI 0 Alt/IMU 1 / IMU 2 --> SPI 1"
- note added: "Battery"

Commit message: added-more-leds
Connections:
- net YELLOW_LED: now reaches A1.D6
- net GREEN_LED: now reaches A1.D7
- net BLUE_LED: now reaches A1.D8
- net LED renamed RED_LED
- no-connect marks 22 -> 19
Changed lines of the file:
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@@
 	(text "Digital"
 		(exclude_from_sim no)
-		(at 226.06 43.18 0)
+		(at 231.14 44.45 0)
 		(effects
 			(font
@@
 	)
 	(no_connect
-		(at 212.09 88.9)
-	)
-	(no_connect
 		(at 212.09 93.98)
 	)
@@
 	)
 	(no_connect
-		(at 212.09 86.36)
-	)
-	(no_connect
 		(at 186.69 96.52)
 	)
@@
 	)
 	(no_connect
-		(at 212.09 83.82)
-	)
-	(no_connect
 		(at 186.69 38.1)
 	)
@@
 		)
 	)
+	(global_label "BLUE_LED"
+		(shape input)
+		(at 212.09 83.82 0)
+		(fields_autoplaced yes)
+		(effects
+			(font
+				(size 1.27 1.27)
+			)
+			(justify left)
+		)
+		(property "Intersheetrefs" "${INTERSHEET_REFS}"
+			(at 224.2675 83.82 0)
+			(hide yes)
+			(show_name no)
+			(do_not_autoplace no)
+			(effects
+				(font
+					(size 1.27 1.27)
+				)
+				(justify left)
+			)
+		)
+	)
 	(global_label "SCK1"
 		(shape input)
@@
 		)
 	)
-	(global_label "LED"
+	(global_label "RED_LED"
 		(shape input)
 		(at 215.9 43.18 0)
@@
 		)
 		(property "Intersheetrefs" "${INTERSHEET_REFS}"
-			(at 222.3323 43.18 0)
+			(at 226.9889 43.18 0)
 			(hide yes)
 			(show_name no)
@@
 		)
 	)
+	(global_label "GREEN_LED"
+		(shape input)
+		(at 212.09 86.36 0)
+		(fields_autoplaced yes)
+		(effects
+			(font
+				(size 1.27 1.27)
+			)
+			(justify left)
+		)
+		(property "Intersheetrefs" "${INTERSHEET_REFS}"
+			(at 225.6584 86.36 0)
+			(hide yes)
+			(show_name no)
+			(do_not_autoplace no)
+			(effects
+				(font
+					(size 1.27 1.27)
+				)
+				(justify left)
+			)
+		)
+	)
 	(global_label "INT_I0"
 		(shape input)
@@
 			(hide yes)
 			(show_name no)
+			(do_not_autoplace no)
+			(effects
+				(font
+					(size 1.27 1.27)
+				)
+				(justify left)
+			)
+		)
+	)
+	(global_label "YELLOW_LED"
+		(shape input)
+		(at 212.09 88.9 0)
+		(fields_autoplaced yes)
+		(effects
+			(font
+				(size 1.27 1.27)
+			)
+			(justify left)
+		)
+		(property "Intersheetrefs" "${INTERSHEET_REFS}"
+			(at 226.5656 88.9 0)
+			(hide yes)
+			(show_name no)

Commit message: simple-fixes
Other:
- note removed: "Alt/IMU 0 / Alt 2 --> SPI 0 Alt/IMU 1 / IMU 2 --> SPI 1"
- note removed: "Digital"
- note removed: "PWM"
- note removed: "interrupts? maybe? no?"
Changed lines of the file:
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@@
 		(company "Notre Dame Rocketry Team")
-	)
-	(text "Alt/IMU 0 / Alt 2 --> SPI 0\nAlt/IMU 1 / IMU 2 --> SPI 1"
-		(exclude_from_sim no)
-		(at 239.395 25.4 0)
-		(effects
-			(font
-				(size 1.27 1.27)
-			)
-		)
-	)
-	(text "PWM"
-		(exclude_from_sim no)
-		(at 227.33 40.64 0)
-		(effects
-			(font
-				(size 1.27 1.27)
-			)
-		)
-	)
-	(text "interrupts? maybe? no?"
-		(exclude_from_sim no)
-		(at 246.38 73.025 0)
-		(effects
-			(font
-				(size 1.27 1.27)
-			)
-		)
 	)
 	(text "Battery"
 		(exclude_from_sim no)
 		(at 210.82 139.7 0)
-		(effects
-			(font
-				(size 1.27 1.27)
-			)
-		)
-	)
-	(text "Digital"
-		(exclude_from_sim no)
-		(at 231.14 44.45 0)
 		(effects
 			(font
@@
 	)
 	(no_connect
+		(at 212.09 35.56)
+	)
+	(no_connect
 		(at 186.69 96.52)
 	)
@@
 	)
 	(no_connect
-		(at 220.345 35.56)
-	)
-	(no_connect
 		(at 186.69 66.04)
 	)
@@
 		(pts
 			(xy 178.435 55.88) (xy 186.69 55.88)
-		)
-		(stroke
-			(width 0)
-			(type default)
-		)
-	)
-	(wire
-		(pts
-			(xy 212.09 35.56) (xy 220.345 35.56)
 		)
 		(stroke
@@
 	)
 	(sheet
-		(at 100.33 159.385)
-		(size 52.07 37.465)
+		(at 97.79 159.385)
+		(size 54.61 37.465)
 		(exclude_from_sim no)
 		(in_bom yes)
@@
 		)
 		(property "Sheetname" "IMUs"
-			(at 100.33 158.6734 0)
+			(at 97.79 158.6734 0)
 			(show_name no)
 			(do_not_autoplace no)
@@
 		)
 		(property "Sheetfile" "acs_IMUs.kicad_sch"
-			(at 100.33 197.4346 0)
-			(show_name no)
-			(do_not_autoplace no)
+			(at 97.79 197.4346 0)
+			(show_name no)
+			(do_not_autoplace no)

Commit message: added power protections
Parts:
- added D5: B540C-13-F, symbol Device:D_Schottky
- added F1: 0685H9100-01, symbol Device:Fuse
Connections:
- net +BATT: now also D5.1 (K), F1.1; no longer J5.1 (Pin_1)
- net GND: now also D5.2 (A)
- new net: F1.2, J5.1 (Pin_1)
Other:
- moved on the sheet: J5

Commit message: miso-mosi-fix
Connections:
- net MISO0: now also A1.D12 ((SDI)D12); no longer A1.D11 ((SDO)D11)
- net MISO1: now also A1.D39 (A15); no longer A1.D26 (A12)
- net MOSI0: now also A1.D11 ((SDO)D11); no longer A1.D12 ((SDI)D12)
- net MOSI1: now also A1.D26 (A12); no longer A1.D39 (A15)
Other:
- note added: "Miso / mosi"
- note added: "Put LCSC part numbers in the values tables"

Commit message: created PCB and layout
Parts:
- A1: footprint Teensy:Teensy41 -> Teensy 4.1:Teensy41
- D5: footprint (none) -> Diode_SMD:D_SMC
- F1: footprint (none) -> Fuse:Fuse_1206_3216Metric
- J5: footprint (none) -> Connector_AMASS:AMASS_XT60-F_1x02_P7.20mm_Vertical
Connections:
- net +3.3V: now also A1.3.3V; no longer A1.3V3 (3.3V)
- net BLUE_LED: now also A1.8 (D8); no longer A1.D8
- net Buzzer: now also A1.33 (D33); no longer A1.D33
- net CS_A0: now also A1.10 ((CS)D10); no longer A1.D10 ((CS)D10)
- net CS_A1: now also A1.14 (A0); no longer A1.D14 (A0)
- net CS_A2: now also A1.16 (A2); no longer A1.D16 (A2)
- net CS_I0: now also A1.9 (D9); no longer A1.D9
- net CS_I1: now also A1.15 (A1); no longer A1.D15 (A1)
- net CS_I2: now also A1.17 (A3); no longer A1.D17 (A3)
- net GND: no longer A1.AGND/GND (GND), A1.GND@2 (GND)
- net GREEN_LED: now also A1.7 (D7); no longer A1.D7
- net INT_A0: now also A1.36 (D36); no longer A1.D36
- net INT_A1: now also A1.32 (D32); no longer A1.D32
- net INT_A2: now also A1.30 (D30); no longer A1.D30
- net INT_I0: now also A1.37 (D37); no longer A1.D37
- net INT_I1: now also A1.31 (D31); no longer A1.D31
- net INT_I2: now also A1.29 (D29); no longer A1.D29
- net MISO0: now also A1.12 ((SDI)D12); no longer A1.D12 ((SDI)D12)
- net MISO1: now also A1.39 (A15); no longer A1.D39 (A15)
- net MOSI0: now also A1.11 ((SDO)D11); no longer A1.D11 ((SDO)D11)
- net MOSI1: now also A1.26 (A12); no longer A1.D26 (A12)
- net PWM_fs: now also A1.24 (A10); no longer A1.D24 (A10)
- net RED_LED: now also A1.5 (D5); no longer A1.D34
- net SCK0: now also A1.13 ((CLK)D13); no longer A1.D13 ((CLK)D13)
- net SCK1: now also A1.27 (A13); no longer A1.D27 (A13)
- net VoltMonitor: now also A1.22 (A8); no longer A1.D28
- net YELLOW_LED: now also A1.6 (D6); no longer A1.D6
- removed net PWM_ss: A1.D25 (A11)
- no-connect marks 19 -> 20
Other:
- note removed: "Miso / mosi"
- note removed: "Put LCSC part numbers in the values tables"
- moved on the sheet: A1

Commit message: voltage converter, PCB setup, battery
Connections:
- net 5V renamed +5V
Changed lines of the file:
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@@
-		)
-	)
-	(global_label "5V"
-		(shape input)
-		(at 219.075 33.02 0)
-		(fields_autoplaced yes)
-		(effects
-			(font
-				(size 1.27 1.27)
-			)
-			(justify left)
-		)
-		(property "Intersheetrefs" "${INTERSHEET_REFS}"
-			(at 224.3583 33.02 0)
-			(hide yes)
-			(show_name no)
-			(do_not_autoplace no)
-			(effects
-				(font
-					(size 1.27 1.27)
-				)
-				(justify left)
-			)
 		)
 	)
@@
 					(unit 1)
 				)
+			)
+		)
+	)
+	(symbol
+		(lib_id "power:+5V")
+		(at 219.075 33.02 270)
+		(unit 1)
+		(body_style 1)
+		(exclude_from_sim no)
+		(in_bom yes)
+		(on_board yes)
+		(in_pos_files yes)
+		(dnp no)
+		(fields_autoplaced yes)
+		(property "Reference" "#PWR016"
+			(at 215.265 33.02 0)
+			(hide yes)
+			(show_name no)
+			(do_not_autoplace no)
+			(effects
+				(font
+					(size 1.27 1.27)
+				)
+			)
+		)
+		(property "Value" "+5V"
+			(at 222.25 33.0199 90)
+			(show_name no)
+			(do_not_autoplace no)
+			(effects
+				(font
+					(size 1.27 1.27)
+				)
+				(justify left)
+			)
+		)
+		(property "Footprint" ""
+			(at 219.075 33.02 0)
+			(hide yes)
+			(show_name no)
+			(do_not_autoplace no)
+			(effects
+				(font
+					(size 1.27 1.27)
+				)
+			)
+		)
+		(property "Datasheet" ""
+			(at 219.075 33.02 0)
+			(hide yes)
+			(show_name no)
+			(do_not_autoplace no)
+			(effects
+				(font
+					(size 1.27 1.27)
+				)
+			)
+		)
+		(property "Description" "Power symbol creates a global label with name \"+5V\""
+			(at 219.075 33.02 0)
+			(hide yes)
+			(show_name no)
+			(do_not_autoplace no)
+			(effects
+				(font
+					(size 1.27 1.27)
+				)
+			)
+		)
+		(pin "1"
+		)
+		(instances
+			(project "ACS PCB"
+				(path "/67a598cb-afc0-4277-b58a-8f35d31efc48"
+					(reference "#PWR016")
+					(unit 1)
+				)
