File: LEDindicator.kicad_sch (KiCad schematic)
At the start: 0 parts

Commit message: Added LED and Passive Buzzers on Indicator sheet. I added the globallabels for connections on the main sheet as well.
Parts:
- added BZ1: Buzzer, Buzzer_Beeper:Buzzer_TDK_PS1240P02BT_D12.2mm_H6.5mm, symbol Device:Buzzer
- added D1: LED, LED_SMD:LED_0805_2012Metric, symbol Device:LED
- added Q1: 2SC1815, Package_TO_SOT_THT:TO-92_Inline, symbol Transistor_BJT:2SC1815
- added R10, R11: 1k, Resistor_SMD:R_0805_2012Metric, symbol Device:R
- added R9: 1K, Resistor_SMD:R_0805_2012Metric, symbol Device:R
Connections:
- new net: D1.1 (K), R9.2
- new net: BZ1.2 (-), Q1.2 (C), R11.2
- new net: Q1.3 (B), R10.2
- new net 3.3V: BZ1.1 (+), R11.1
- new net Buzzer: R10.1
- new net GND: D1.2 (A), Q1.1 (E)
- new net LED: R9.1
Other:
- note added: "Buzzer Indicator"
- note added: "LED Indicator"
