File: LEDindicator.kicad_sch (KiCad schematic)
At the start: 6 parts, among them Q1 2SC1815

Commit message: Fixed symbols and ran ERC
Other:
- note added: "Indicators"
Changed lines of the file:
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@@
+		)
+	)
+	(text "Indicators"
+		(exclude_from_sim no)
+		(at 132.715 32.385 0)
+		(effects
+			(font
+				(size 6.35 6.35)
+			)
 		)
 	)

Commit message: added-more-leds
Parts:
- added D2, D3, D4: LED, LED_SMD:LED_0805_2012Metric, symbol Device:LED
- added R14, R15, R16: 1K, Resistor_SMD:R_0805_2012Metric, symbol Device:R
Connections:
- net GND: now also D2.2 (A), D3.2 (A), D4.2 (A)
- net LED renamed RED_LED
- new net: D4.1 (K), R16.2
- new net: D2.1 (K), R14.2
- new net: D3.1 (K), R15.2
- new net BLUE_LED: R15.1
- new net GREEN_LED: R16.1
- new net YELLOW_LED: R14.1
Other:
- note added: "BLUE LED Indicator"
- note added: "GREEN LED Indicator"
- note added: "RED LED Indicator"
- note added: "YELLOW LED Indicator"
- note removed: "LED Indicator"
- moved on the sheet: D1, R9

Commit message: simple-fixes
Connections:
- net GND: now also D1.1 (K), D2.1 (K), D3.1 (K), D4.1 (K); no longer D1.2 (A), D2.2 (A), D3.2 (A), D4.2 (A)
- net at R9.2: now also D1.2 (A); no longer D1.1 (K)
- net at R16.2: now also D4.2 (A); no longer D4.1 (K)
- net at R14.2: now also D2.2 (A); no longer D2.1 (K)
- net at R15.2: now also D3.2 (A); no longer D3.1 (K)
Other:
- moved on the sheet: D1, D2, D3, D4
Changed lines of the file:
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@@
 	(symbol
 		(lib_id "Device:LED")
-		(at 102.87 123.19 0)
+		(at 102.87 123.19 180)
 		(unit 1)
 		(body_style 1)
@@
 		(fields_autoplaced yes)
 		(property "Reference" "D4"
-			(at 101.2825 116.84 0)
+			(at 104.4575 115.57 0)
 			(show_name no)
 			(do_not_autoplace no)
@@
 		)
 		(property "Value" "LED"
-			(at 101.2825 119.38 0)
+			(at 104.4575 118.11 0)
 			(show_name no)
 			(do_not_autoplace no)
@@
 	(symbol
 		(lib_id "Device:LED")
-		(at 102.87 86.36 0)
+		(at 102.87 86.36 180)
 		(unit 1)
 		(body_style 1)
@@
 		(fields_autoplaced yes)
 		(property "Reference" "D2"
-			(at 101.2825 80.01 0)
+			(at 104.4575 78.74 0)
 			(show_name no)
 			(do_not_autoplace no)
@@
 		)
 		(property "Value" "LED"
-			(at 101.2825 82.55 0)
+			(at 104.4575 81.28 0)
 			(show_name no)
 			(do_not_autoplace no)
@@
 	(symbol
 		(lib_id "Device:LED")
-		(at 102.87 66.04 0)
+		(at 102.87 66.04 180)
 		(unit 1)
 		(body_style 1)
@@
 		(fields_autoplaced yes)
 		(property "Reference" "D1"
-			(at 101.2825 59.69 0)
+			(at 104.4575 58.42 0)
 			(show_name no)
 			(do_not_autoplace no)
@@
 		)
 		(property "Value" "LED"
-			(at 101.2825 62.23 0)
+			(at 104.4575 60.96 0)
 			(show_name no)
 			(do_not_autoplace no)
@@
 	(symbol
 		(lib_id "Device:LED")
-		(at 102.87 104.14 0)
+		(at 102.87 104.14 180)
 		(unit 1)
 		(body_style 1)
@@
 		(fields_autoplaced yes)
 		(property "Reference" "D3"
-			(at 101.2825 97.79 0)
+			(at 104.4575 96.52 0)
 			(show_name no)
 			(do_not_autoplace no)
@@
 		)
 		(property "Value" "LED"
-			(at 101.2825 100.33 0)
-			(show_name no)
-			(do_not_autoplace no)
+			(at 104.4575 99.06 0)
+			(show_name no)
+			(do_not_autoplace no)

Commit message: resistor-fix
Parts:
- R10: value 1k -> 10k
Changed lines of the file:
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@@
 			)
 		)
-		(property "Value" "1k"
+		(property "Value" "10k"
 			(at 187.96 100.33 90)
 			(show_name no)

Commit message: Finished up PCB [DRAFT]
Connections:
- net 3.3V renamed +3.3V
Changed lines of the file:
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@@
 		)
 	)
-	(global_label "3.3V"
+	(global_label "GREEN_LED"
 		(shape input)
-		(at 200.66 74.93 90)
+		(at 80.01 123.19 180)
 		(fields_autoplaced yes)
 		(effects
@@
 				(size 1.27 1.27)
 			)
-			(justify left)
+			(justify right)
 		)
 		(property "Intersheetrefs" "${INTERSHEET_REFS}"
-			(at 200.66 67.8324 90)
-			(hide yes)
-			(show_name no)
-			(do_not_autoplace no)
-			(effects
-				(font
-					(size 1.27 1.27)
-				)
-				(justify left)
-			)
-		)
-	)
-	(global_label "GREEN_LED"
+			(at 66.4416 123.19 0)
+			(hide yes)
+			(show_name no)
+			(do_not_autoplace no)
+			(effects
+				(font
+					(size 1.27 1.27)
+				)
+				(justify right)
+			)
+		)
+	)
+	(global_label "BLUE_LED"
 		(shape input)
-		(at 80.01 123.19 180)
+		(at 80.01 104.14 180)
 		(fields_autoplaced yes)
 		(effects
@@
 		)
 		(property "Intersheetrefs" "${INTERSHEET_REFS}"
-			(at 66.4416 123.19 0)
+			(at 67.8325 104.14 0)
 			(hide yes)
 			(show_name no)
@@
 		)
 	)
-	(global_label "BLUE_LED"
+	(global_label "Buzzer"
 		(shape input)
-		(at 80.01 104.14 180)
+		(at 182.88 104.14 180)
 		(fields_autoplaced yes)
 		(effects
@@
 		)
 		(property "Intersheetrefs" "${INTERSHEET_REFS}"
-			(at 67.8325 104.14 0)
+			(at 173.5448 104.14 0)
 			(hide yes)
 			(show_name no)
@@
 		)
 	)
-	(global_label "Buzzer"
+	(global_label "RED_LED"
 		(shape input)
-		(at 182.88 104.14 180)
+		(at 80.01 66.04 180)
 		(fields_autoplaced yes)
 		(effects
@@
 		)
 		(property "Intersheetrefs" "${INTERSHEET_REFS}"
-			(at 173.5448 104.14 0)
+			(at 68.9211 66.04 0)
 			(hide yes)
 			(show_name no)
@@
 		)
 	)
-	(global_label "RED_LED"
+	(global_label "YELLOW_LED"
 		(shape input)
-		(at 80.01 66.04 180)
+		(at 80.01 86.36 180)
 		(fields_autoplaced yes)
 		(effects
@@
 		)
 		(property "Intersheetrefs" "${INTERSHEET_REFS}"
-			(at 68.9211 66.04 0)
-			(hide yes)
-			(show_name no)
-			(do_not_autoplace no)
-			(effects
-				(font
-					(size 1.27 1.27)
-				)
-				(justify right)
-			)
-		)
-	)
-	(global_label "YELLOW_LED"
-		(shape input)
-		(at 80.01 86.36 180)
-		(fields_autoplaced yes)
-		(effects
-			(font
-				(size 1.27 1.27)
-			)
-			(justify right)
-		)
-		(property "Intersheetrefs" "${INTERSHEET_REFS}"
 			(at 65.5344 86.36 0)
 			(hide yes)
@@
 					(unit 1)
 				)
+			)
+		)
+	)
+	(symbol
+		(lib_id "power:+3.3V")
+		(at 200.66 74.93 0)
+		(unit 1)
+		(body_style 1)
+		(exclude_from_sim no)
+		(in_bom yes)
+		(on_board yes)
+		(in_pos_files yes)
+		(dnp no)
+		(fields_autoplaced yes)
+		(property "Reference" "#PWR017"
+			(at 200.66 78.74 0)
+			(hide yes)
+			(show_name no)
+			(do_not_autoplace no)
+			(effects
+				(font
+					(size 1.27 1.27)
+				)
+			)
+		)
+		(property "Value" "+3.3V"
+			(at 200.66 69.85 0)
+			(show_name no)
+			(do_not_autoplace no)
+			(effects
+				(font
+					(size 1.27 1.27)
+				)
+			)
+		)
+		(property "Footprint" ""
+			(at 200.66 74.93 0)
+			(hide yes)
+			(show_name no)
+			(do_not_autoplace no)
+			(effects
+				(font
+					(size 1.27 1.27)
+				)
+			)
+		)
+		(property "Datasheet" ""
+			(at 200.66 74.93 0)
+			(hide yes)
+			(show_name no)
+			(do_not_autoplace no)
+			(effects
+				(font
+					(size 1.27 1.27)
+				)
+			)
+		)
+		(property "Description" "Power symbol creates a global label with name \"+3.3V\""
+			(at 200.66 74.93 0)
+			(hide yes)
+			(show_name no)
+			(do_not_autoplace no)
+			(effects
+				(font
+					(size 1.27 1.27)
+				)
+			)
+		)
+		(pin "1"
+		)
+		(instances
+			(project "ACS PCB"
+				(path "/67a598cb-afc0-4277-b58a-8f35d31efc48/52e21e5d-46e6-440d-b2c7-d7be369a43cb"
+					(reference "#PWR017")
+					(unit 1)
+				)

Commit message: Redid Footprints/Picked components
Parts:
- R14, R15, R16, R9: value 1K -> 1k
Changed lines of the file:
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@@
 			)
 		)
-		(property "Value" "1K"
+		(property "Value" "1k"
 			(at 91.44 62.23 90)
 			(show_name no)
@@
 			)
 		)
-		(property "Value" "1K"
+		(property "Value" "1k"
 			(at 91.44 119.38 90)
 			(show_name no)
@@
 			)
 		)
-		(property "Value" "1K"
+		(property "Value" "1k"
 			(at 91.44 82.55 90)
 			(show_name no)
@@
 			)
 		)
-		(property "Value" "1K"
+		(property "Value" "1k"
 			(at 91.44 100.33 90)
 			(show_name no)
