File: acs_IMUs.kicad_sch (KiCad schematic)
At the start: 9 parts, among them U1 LSM6DSV80XTR, U3 LSM6DSV80XTR, U7 LSM6DSV80XTR

Commit message: Fixed symbols and ran ERC
Parts:
- U1, U3, U7: footprint QFN_LSM6DSV80XTR_STM -> LSM6DSV80XTR:QFN_LSM6DSV80XTR_STM
Connections:
- net VDDIO is gone; now on net +3.3V: C13.1, C15.1, C17.1, U1.5 (VDDIO), U3.5 (VDDIO), U7.5 (VDDIO)
- net CS1 renamed CS_I0
- net CS3 renamed CS_I1
- net CS7 renamed CS_I2
- net INT1 renamed INT_I0
- net INT3 renamed INT_I1
- net INT7 renamed INT_I2
- net SCK renamed SCK1
- net SCK1: no longer U1.13 (SCL)
- net SDI renamed MOSI1
- net MOSI1: no longer U1.14 (SDA)
- net SDO renamed MISO1
- net MISO1: no longer U1.1 (SDO)
- net VDD renamed +3.3V
- new net MISO0: U1.1 (SDO)
- new net MOSI0: U1.14 (SDA)
- new net SCK0: U1.13 (SCL)
Other:
- note added: "IMU"
- note added: "IMU 0"
- note added: "IMU 1"
- note added: "IMU 2(1)"
- moved on the sheet: C13, C14, U1

Commit message: added power protections
Parts:
- added R1, R13, R17, R18, R19, R2: 10R, symbol Device:R_US
Connections:
- net +3.3V: now also R1.1, R13.1, R17.2, R18.2, R19.1, R2.2; no longer C13.1, C14.1, C15.1, C16.1, C17.1, C18.1, U1.5 (VDDIO), U1.8 (VDD), U3.5 (VDDIO), U3.8 (VDD), U7.5 (VDDIO), U7.8 (VDD)
- new net: C18.1, R18.1, U7.8 (VDD)
- new net: C13.1, R1.2, U1.5 (VDDIO)
- new net: C15.1, R13.2, U3.5 (VDDIO)
- new net: C17.1, R19.2, U7.5 (VDDIO)
- new net: C16.1, R17.1, U3.8 (VDD)
- new net: C14.1, R2.1, U1.8 (VDD)
Other:
- moved on the sheet: C15, C16, C17, C18, U3, U7

Commit message: miso-mosi-fix
Parts:
- R1, R13, R17, R18, R19, R2: footprint (none) -> Resistor_SMD:R_0603_1608Metric
Other:
- moved on the sheet: C13, C15
