File: motorInterfacing.kicad_sch (KiCad schematic)
At the start: 6 parts, among them J1 Conn_01x02, J2 Conn_01x02, J3 Conn_01x01, J4 Conn_01x01

Commit message: miso-mosi-fix
Parts:
- C21, C25: footprint (none) -> Capacitor_SMD:C_0603_1608Metric
Other:
- note added: "Make sure capacitors are rated"
Changed lines of the file:
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@@
 		(company "Notre Dame Rocketry Team")
+	)
+	(text "Make sure capacitors are rated"
+		(exclude_from_sim no)
+		(at 106.045 107.95 0)
+		(effects
+			(font
+				(size 1.27 1.27)
+			)
+		)
 	)
 	(text "DS51150 — Fullscale  Motor"
@@
 			)
 		)
-		(property "Footprint" ""
+		(property "Footprint" "Capacitor_SMD:C_0603_1608Metric"
 			(at 92.075 76.835 0)
 			(hide yes)
@@
 			)
 		)
-		(property "Footprint" ""
+		(property "Footprint" "Capacitor_SMD:C_0603_1608Metric"
 			(at 210.82 72.39 0)
 			(hide yes)
