File: ACS PCB.kicad_pcb (KiCad board)
At the start: 4 copper layers, 72.4 x 72.4 mm, 64 parts, among them J1 Conn_01x02, J3 Conn_01x01, J5 Conn_01x02, Q1 2SC1815, U1 LSM6DSV80XTR, U3 LSM6DSV80XTR, U4 BMP581, U5 BMP581, U6 BMP581, U7 LSM6DSV80XTR, U8 PLM62440APPQRJRTQ1

Commit message: voltage converter, PCB setup, battery
Parts:
- moved C20 4.51 mm to (131.1, 69.4)
- moved C2 3.20 mm to (131.1, 72.5)
- moved L1 3.15 mm to (131.1, 74.0)
- moved F1 3.01 mm to (139.3, 65.8)
- moved D5 2.99 mm to (146.8, 68.0)
- moved C22 1.46 mm to (131.1, 70.9)
- moved C4 0.33 mm to (122.8, 75.5)
- moved C5 0.33 mm to (122.8, 73.9)
- moved R12 0.33 mm to (122.7, 77.1)
Connections:
- A1 pad VIN: 5V -> +5V
Routing:
- net +BATT: track 0.00 -> 73.4 mm, vias 0 -> 3
- net +5V: track 0.00 -> 31.6 mm, vias 0 -> 2
- net Net-(U8-CBOOT): track 0.00 -> 15.1 mm, vias 0 -> 2
- net Net-(J5-Pin_1): track 0.00 -> 14.8 mm, vias 0 -> 1
- net Net-(U8-MODE_SYNC): track 0.00 -> 4.43 mm
- net Net-(U8-SW): track 0.00 -> 3.86 mm
- net +3.3V: track 0.00 -> 3.63 mm
- added copper zone on In2.Cu, net (none)
- added copper zone on In2.Cu, net +3.3V
- added copper zone on In2.Cu, net +5V
- added copper zone on In2.Cu, net GND

Commit message: routing for IMUs
Routing:
- net CS_I1: track 0.00 -> 39.9 mm
- net INT_I0: track 0.00 -> 37.8 mm, vias 0 -> 1
- net MISO1: track 0.00 -> 33.4 mm
- net CS_I2: track 0.00 -> 30.1 mm, vias 0 -> 2
- net SCK0: track 0.00 -> 24.2 mm, vias 0 -> 1
- net INT_I2: track 0.00 -> 19.0 mm, vias 0 -> 1
- net SCK1: track 0.00 -> 15.8 mm, vias 0 -> 1
- net MOSI1: track 0.00 -> 15.8 mm, vias 0 -> 1
- net INT_I1: track 0.00 -> 12.5 mm, vias 0 -> 1
- net MISO0: track 0.00 -> 11.4 mm, vias 0 -> 1
- net MOSI0: track 0.00 -> 7.32 mm
- net CS_I0: track 0.00 -> 6.07 mm, vias 0 -> 1
- net Net-(U7-VDDIO): track 0.00 -> 3.55 mm
- net Net-(U1-VDD): track 0.00 -> 3.48 mm
- net Net-(U3-VDD): track 0.00 -> 3.46 mm
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
Commit message: Traced LED
Routing:
- net BLUE_LED: track 0.00 -> 14.9 mm
- net YELLOW_LED: track 0.00 -> 13.3 mm
- net GREEN_LED: track 0.00 -> 9.59 mm, vias 0 -> 1
- net RED_LED: track 0.00 -> 9.13 mm
- net GND: track 0.00 -> 9.09 mm, vias 0 -> 2
- net Net-(D4-A): track 0.00 -> 7.00 mm
- net Net-(D3-A): track 0.00 -> 4.36 mm
- net Net-(D1-A): track 0.00 -> 4.35 mm
- net Net-(D2-A): track 0.00 -> 4.34 mm
