File: power.kicad_sch (KiCad schematic)
At the start: 9 parts, among them U2 TPSM84338RCJR

Commit message: power convertor
Parts:
- added C19, C20, C21, C22, C23, C24, C25: C, symbol Device:C
- added L1: L, symbol Device:L
- added R12, R13, R14, R15: R_US, symbol Device:R_US
- added U8: PLM62440APPQRJRTQ1, LM6440:RJR0014A-MFG, symbol LM62440:PLM62440APPQRJRTQ1
Connections:
- net GND: now also C19.2, C20.2, C21.2, C23.2, C25.2, R14.2, U8.11 (PGND2), U8.3 (AGND), U8.6 (MODE_SYNC), U8.9 (PGND1)
- net Vin: now also C23.1, L1.2, R12.2, R13.1, R15.1, U8.1 (BIAS)
- new net: C24.2, R13.2, R14.1, U8.4 (FB)
- new net: C24.1, R15.2
- new net: C22.1, L1.1, U8.10 (SW)
- new net: C22.2, U8.13 (RBOOT), U8.14 (CBOOT)
- new net: R12.1, U8.5 (PGOOD)
- new net: C25.1, U8.2 (VCC)
- new net +BATT: C19.1, C20.1, C21.1, U8.12 (VIN2), U8.7 (EN), U8.8 (VIN1)
Other:
- note added: "have not done footprints yet!!"
- moved on the sheet: C1, C2, C3, C4, C5, C6, R1, R2, U2

Commit message: finished voltage converter i think :sob: ugh ugh ughgit add .git add .
Parts:
- removed C2: 10u, Capacitor_SMD:C_0603_1608Metric, symbol Device:C
- removed C3, C6: 100n, Capacitor_SMD:C_0603_1608Metric, symbol Device:C
- removed C4, C5: 22u, Capacitor_SMD:C_0603_1608Metric, symbol Device:C
- removed R1: 30k, Resistor_SMD:R_0603_1608Metric, symbol Device:R_US
- removed R14, R15: R_US, symbol Device:R_US
- removed R2: 220k, Resistor_SMD:R_0603_1608Metric, symbol Device:R_US
- removed U2: TPSM84338RCJR, RCJ0009A-MFG, symbol TPSM84338RCJR:TPSM84338RCJR
- added C26, C27: 22uF, Capacitor_SMD:C_0603_1608Metric, symbol Device:C
- added C28: 10uF, symbol Device:C
- C1: value 10u -> 100uF; footprint Capacitor_SMD:C_0603_1608Metric -> (none)
- C19, C25: value C -> 22uF; footprint (none) -> Capacitor_SMD:C_0603_1608Metric
- C20: value C -> 1uF
- C21, C22, C23: value C -> 100nF
- C24: value C -> 10uF
- L1: value L -> 4.7uH
- R12: value R_US -> 10k
- R13: value R_US -> 0R
- U8: footprint LM6440:RJR0014A-MFG -> RJR0014A-MFG
Connections:
- net +BATT: now also C1.2, C22.1, C24.1, C28.1; no longer C19.1, C20.1
- net GND: now also C22.2, C24.2, C26.2, C27.2, C28.2; no longer C23.2, U8.6 (MODE_SYNC)
- net at L1.1, U8.10 (SW): now also C23.1; no longer C22.1
- net VoltMonitor: now reaches R12.1, U8.5 (PGOOD)
- net at U8.2 (VCC): now also C20.1, U8.6 (MODE_SYNC); no longer C25.1
- removed net Vin: C1.2, C23.1, L1.2, R12.2, R13.1, U8.1 (BIAS)
- new net: C23.2, R13.1, U8.14 (CBOOT)
- new net: R13.2, U8.13 (RBOOT)
- new net 3.3V: R12.2
- new net 5V: C19.1, C25.1, C26.1, C27.1, L1.2, U8.1 (BIAS), U8.4 (FB)
- no-connect marks 5 -> 0
Other:
- note added: ":("
- note removed: "apparently ts bad :("
- note removed: "have not done footprints yet!!"
- note removed: "should be >25V rated capacitors"

Commit message: Fixed symbols and ran ERC
Parts:
- C1: footprint (none) -> Capacitor_SMD:C_0201_0603Metric
- U8: footprint RJR0014A-MFG -> LM6440:RJR0014A-MFG
Other:
- note added: "Power"
- note removed: ":("
Changed lines of the file:
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@@
 		(company "Notre Dame Rocketry Team")
 	)
-	(text ":("
+	(text "Power"
 		(exclude_from_sim no)
-		(at 116.84 36.83 0)
+		(at 152.4 28.575 0)
 		(effects
 			(font
-				(size 1.27 1.27)
+				(size 6.35 6.35)
 			)
 		)
@@
 	)
 	(junction
+		(at 89.535 84.455)
+		(diameter 0)
+		(color 0 0 0 0)
+	)
+	(junction
 		(at 201.295 81.915)
 		(diameter 0)
@@
 	(wire
 		(pts
+			(xy 89.535 84.455) (xy 93.98 84.455)
+		)
+		(stroke
+			(width 0)
+			(type default)
+		)
+	)
+	(wire
+		(pts
 			(xy 201.295 94.615) (xy 215.9 94.615)
 		)
@@
 	(wire
 		(pts
-			(xy 85.09 84.455) (xy 93.98 84.455)
+			(xy 85.09 84.455) (xy 89.535 84.455)
 		)
 		(stroke
@@
 			)
 		)
-		(property "Footprint" "RJR0014A-MFG"
+		(property "Footprint" "LM6440:RJR0014A-MFG"
 			(at 93.98 61.595 0)
 			(hide yes)
@@
 	)
 	(symbol
+		(lib_id "power:PWR_FLAG")
+		(at 89.535 84.455 180)
+		(unit 1)
+		(body_style 1)
+		(exclude_from_sim no)
+		(in_bom yes)
+		(on_board yes)
+		(in_pos_files yes)
+		(dnp no)
+		(fields_autoplaced yes)
+		(property "Reference" "#FLG03"
+			(at 89.535 86.36 0)
+			(hide yes)
+			(show_name no)
+			(do_not_autoplace no)
+			(effects
+				(font
+					(size 1.27 1.27)
+				)
+			)
+		)
+		(property "Value" "PWR_FLAG"
+			(at 89.535 88.9 0)
+			(show_name no)
+			(do_not_autoplace no)
+			(effects
+				(font
+					(size 1.27 1.27)
+				)
+			)
+		)
+		(property "Footprint" ""
+			(at 89.535 84.455 0)
+			(hide yes)
+			(show_name no)
+			(do_not_autoplace no)
+			(effects
+				(font
+					(size 1.27 1.27)
+				)
+			)
+		)
+		(property "Datasheet" ""
+			(at 89.535 84.455 0)
+			(hide yes)
+			(show_name no)
+			(do_not_autoplace no)
+			(effects
+				(font
+					(size 1.27 1.27)
+				)
+			)
+		)
+		(property "Description" "Special symbol for telling ERC where power comes from"
+			(at 89.535 84.455 0)
+			(hide yes)
+			(show_name no)
+			(do_not_autoplace no)
+			(effects
+				(font
+					(size 1.27 1.27)
+				)
+			)
+		)
+		(pin "1"
+		)
+		(instances
+			(project "ACS PCB"
+				(path "/67a598cb-afc0-4277-b58a-8f35d31efc48/8f3a2ae2-24ee-4ca8-930f-6202803bc7c8"
+					(reference "#FLG03")
+					(unit 1)
+				)
+			)
+		)
+	)
+	(symbol
 		(lib_id "power:+BATT")
 		(at 52.07 50.165 90)
@@
 			)
 		)
-		(property "Footprint" ""
+		(property "Footprint" "Capacitor_SMD:C_0201_0603Metric"
 			(at 54.2798 56.515 0)
 			(hide yes)

Commit message: i think i fixed it??
Connections:
- net 3.3V renamed +3.3V
- net 5V renamed +5V
Changed lines of the file:
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@@
+	)
+	(junction
+		(at 247.65 81.915)
+		(diameter 0)
+		(color 0 0 0 0)
 	)
 	(junction
@@
 	(wire
 		(pts
-			(xy 241.935 81.915) (xy 250.19 81.915)
+			(xy 241.935 81.915) (xy 247.65 81.915)
+		)
+		(stroke
+			(width 0)
+			(type default)
+		)
+	)
+	(wire
+		(pts
+			(xy 247.65 81.915) (xy 250.19 81.915)
 		)
 		(stroke
@@
 		)
 	)
-	(global_label "5V"
-		(shape input)
-		(at 250.19 81.915 0)
+	(symbol
+		(lib_id "power:+3.3V")
+		(at 202.565 62.23 270)
+		(unit 1)
+		(body_style 1)
+		(exclude_from_sim no)
+		(in_bom yes)
+		(on_board yes)
+		(in_pos_files yes)
+		(dnp no)
 		(fields_autoplaced yes)
-		(effects
-			(font
-				(size 1.27 1.27)
-			)
-			(justify left)
-		)
-		(property "Intersheetrefs" "${INTERSHEET_REFS}"
-			(at 255.4733 81.915 0)
-			(hide yes)
+		(property "Reference" "#PWR033"
+			(at 198.755 62.23 0)
+			(hide yes)
+			(show_name no)
+			(do_not_autoplace no)
+			(effects
+				(font
+					(size 1.27 1.27)
+				)
+			)
+		)
+		(property "Value" "+3.3V"
+			(at 205.74 62.2299 90)
 			(show_name no)
 			(do_not_autoplace no)
@@
 			)
 		)
-	)
-	(global_label "3.3V"
-		(shape input)
-		(at 202.565 62.23 0)
-		(fields_autoplaced yes)
-		(effects
-			(font
-				(size 1.27 1.27)
-			)
-			(justify left)
-		)
-		(property "Intersheetrefs" "${INTERSHEET_REFS}"
-			(at 209.6626 62.23 0)
-			(hide yes)
-			(show_name no)
-			(do_not_autoplace no)
-			(effects
-				(font
-					(size 1.27 1.27)
-				)
-				(justify left)
+		(property "Footprint" ""
+			(at 202.565 62.23 0)
+			(hide yes)
+			(show_name no)
+			(do_not_autoplace no)
+			(effects
+				(font
+					(size 1.27 1.27)
+				)
+			)
+		)
+		(property "Datasheet" ""
+			(at 202.565 62.23 0)
+			(hide yes)
+			(show_name no)
+			(do_not_autoplace no)
+			(effects
+				(font
+					(size 1.27 1.27)
+				)
+			)
+		)
+		(property "Description" "Power symbol creates a global label with name \"+3.3V\""
+			(at 202.565 62.23 0)
+			(hide yes)
+			(show_name no)
+			(do_not_autoplace no)
+			(effects
+				(font
+					(size 1.27 1.27)
+				)
+			)
+		)
+		(pin "1"
+		)
+		(instances
+			(project "ACS PCB"
+				(path "/67a598cb-afc0-4277-b58a-8f35d31efc48/8f3a2ae2-24ee-4ca8-930f-6202803bc7c8"
+					(reference "#PWR033")
+					(unit 1)
+				)
 			)
 		)
@@
 	)
 	(symbol
+		(lib_id "power:PWR_FLAG")
+		(at 247.65 81.915 0)
+		(unit 1)
+		(body_style 1)
+		(exclude_from_sim no)
+		(in_bom yes)
+		(on_board yes)
+		(in_pos_files yes)
+		(dnp no)
+		(fields_autoplaced yes)
+		(property "Reference" "#FLG011"
+			(at 247.65 80.01 0)
+			(hide yes)
+			(show_name no)
+			(do_not_autoplace no)
+			(effects
+				(font
+					(size 1.27 1.27)
+				)
+			)
+		)
+		(property "Value" "PWR_FLAG"
+			(at 247.65 77.47 0)
+			(show_name no)
+			(do_not_autoplace no)
+			(effects
+				(font
+					(size 1.27 1.27)
+				)
+			)
+		)
+		(property "Footprint" ""
+			(at 247.65 81.915 0)
+			(hide yes)
+			(show_name no)
+			(do_not_autoplace no)
+			(effects
+				(font
+					(size 1.27 1.27)
+				)
+			)
+		)
+		(property "Datasheet" ""
+			(at 247.65 81.915 0)
+			(hide yes)
+			(show_name no)
+			(do_not_autoplace no)
+			(effects
+				(font
+					(size 1.27 1.27)
+				)
+			)
+		)
+		(property "Description" "Special symbol for telling ERC where power comes from"
+			(at 247.65 81.915 0)
+			(hide yes)
+			(show_name no)
+			(do_not_autoplace no)
+			(effects
+				(font
+					(size 1.27 1.27)
+				)
+			)
+		)
+		(pin "1"
+		)
+		(instances
+			(project "ACS PCB"
+				(path "/67a598cb-afc0-4277-b58a-8f35d31efc48/8f3a2ae2-24ee-4ca8-930f-6202803bc7c8"
+					(reference "#FLG011")
+					(unit 1)
+				)
+			)
+		)
+	)
+	(symbol
 		(lib_id "Device:C")
 		(at 159.385 58.42 0)
@@
 					(unit 1)
 				)
+			)
+		)
+	)
+	(symbol
+		(lib_id "power:+5V")
+		(at 250.19 81.915 270)
+		(unit 1)
+		(body_style 1)
+		(exclude_from_sim no)
+		(in_bom yes)
+		(on_board yes)
+		(in_pos_files yes)
+		(dnp no)
+		(fields_autoplaced yes)
+		(property "Reference" "#PWR034"
+			(at 246.38 81.915 0)
+			(hide yes)
+			(show_name no)
+			(do_not_autoplace no)
+			(effects
+				(font
+					(size 1.27 1.27)
+				)
+			)
+		)
+		(property "Value" "+5V"
+			(at 254 81.9149 90)
+			(show_name no)
+			(do_not_autoplace no)
+			(effects
+				(font
+					(size 1.27 1.27)
+				)
+				(justify left)
+			)
+		)
+		(property "Footprint" ""
+			(at 250.19 81.915 0)
+			(hide yes)
+			(show_name no)
+			(do_not_autoplace no)
+			(effects
+				(font
+					(size 1.27 1.27)
+				)
+			)
+		)
+		(property "Datasheet" ""
+			(at 250.19 81.915 0)
+			(hide yes)
+			(show_name no)
+			(do_not_autoplace no)
+			(effects
+				(font
+					(size 1.27 1.27)
+				)
+			)
+		)
+		(property "Description" "Power symbol creates a global label with name \"+5V\""
+			(at 250.19 81.915 0)
+			(hide yes)
+			(show_name no)
+			(do_not_autoplace no)
+			(effects
+				(font
+					(size 1.27 1.27)
+				)
+			)
+		)
+		(pin "1"
+		)
+		(instances
+			(project "ACS PCB"
+				(path "/67a598cb-afc0-4277-b58a-8f35d31efc48/8f3a2ae2-24ee-4ca8-930f-6202803bc7c8"
+					(reference "#PWR034")
+					(unit 1)
+				)

Commit message: simple-fixes
Parts:
- removed C1: 100uF, Capacitor_SMD:C_0201_0603Metric, symbol Device:C
- removed C19, C25, C26, C27: 22uF, Capacitor_SMD:C_0603_1608Metric, symbol Device:C
- removed C20: 1uF, symbol Device:C
- removed C21, C22, C23: 100nF, symbol Device:C
- removed C24, C28: 10uF, symbol Device:C
- removed L1: 4.7uH, symbol Device:L
- removed R13: 0R, symbol Device:R_US
- added C1, C22: 10uF, Capacitor_SMD:C_0603_1608Metric, symbol Device:C_Small
- added C19: 1uF, Capacitor_SMD:C_0603_1608Metric, symbol Device:C_Small
- added C2, C20, C24: 100nF, Capacitor_SMD:C_0603_1608Metric, symbol Device:C_Small
- added C23: 100uF, Capacitor_SMD:C_0603_1608Metric, symbol Device:C_Small
- added C3, C4, C5, C6: 22uF, Capacitor_SMD:C_0603_1608Metric, symbol Device:C_Small
- added L1: 4.7uH, Inductor_SMD:L_0603_1608Metric, symbol Device:L_Small
- R12: footprint (none) -> Resistor_SMD:R_0603_1608Metric
Connections:
- net +5V: now also C3.1, C4.1, C5.1, C6.1, L1.2
- net +BATT: now also C1.1, C20.1, C22.1, C23.1, C24.1
- net GND: now also C1.2, C19.2, C20.2, C22.2, C23.2, C24.2, C3.2, C4.2, C5.2, C6.2
- net at U8.14 (CBOOT): now also U8.13 (RBOOT), C2.2
- net at U8.10 (SW): now also C2.1, L1.1
- net at U8.2 (VCC), U8.6 (MODE_SYNC): now also C19.1
Other:
- moved on the sheet: R12

Commit message: miso-mosi-fix
Changed lines of the file:
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@@
 		(in_pos_files yes)
 		(dnp no)
-		(fields_autoplaced yes)
 		(property "Reference" "L1"
-			(at 153.67 76.835 90)
+			(at 153.67 77.47 90)
 			(show_name no)
 			(do_not_autoplace no)

Commit message: Finished up PCB [DRAFT]
Parts:
- removed L1: 4.7uH, Inductor_SMD:L_0603_1608Metric, symbol Device:L_Small
- added L1: 1090_78439369047, Inductor78439358047:L_Wurth_WE-XHMA-1090, symbol Inductor78439358047:1090_78439369047
Connections:
- net +5V: now also L1.2
- net at C2.1, U8.10 (SW): now also L1.1
Other:
- note added: "WHERE DOES C23 GO????"
